File: kicad/SuperEMUZ80.kicad_pcb (KiCad board)
At the start: 2 copper layers, 99.1 x 76.2 mm, 73 parts, among them J1 Conn_02x01, J11 Conn_02x01, J2 Conn_01x08_Pin, J3 SD Card slot, J4 SD Card slot, J5 5077CR-16SMC2-BK-TR, U1 Z80CPU, U2 18F47Q43, U3 AS6C4008, U4 PIC16F1454-IP

Commit message: Add SuperEMUZ80 version 1.0
Parts:
- added R34: 5k1, Resistor_SMD:R_0603_1608Metric_Pad0.98x0.95mm_HandSolder, F.Cu at (44.3, 91.4)
- added R35: 5k1, Resistor_SMD:R_0603_1608Metric_Pad0.98x0.95mm_HandSolder, F.Cu at (44.5, 88.9)
- D1, D7: value DISK -> LED
- D2, D8: value M1 -> LED
- D3, D9: value POWER -> LED
- D6: value PROG -> LED
- R28, R29: value 220 -> 100
- R30, R32: value 40K -> 39K
- moved C13 0.90 mm to (49.5, 71.1)
Connections:
- J11 pad 2: PIC_RX -> Net-(D4-K)
Routing:
- net Net-(D4-K): track 7.91 -> 37.5 mm, vias 0 -> 1
- net GND: track 344.4 -> 351.2 mm, vias 9 -> 390
- net Net-(J5-CC1): track 6.03 -> 9.68 mm, vias 0 -> 1
- net Net-(J5-CC2): track 5.79 -> 8.58 mm
- net VUSB3V3: track 6.83 -> 4.13 mm, vias 1 -> 0
- net RA4: track 42.9 -> 45.3 mm
- net RA5: track 43.5 -> 45.7 mm
- net LED: track 66.5 -> 67.5 mm
- net ~{MCLR}: track 72.5 -> 71.8 mm
- added copper zone on B.Cu, net GND
- added copper zone on F.Cu, net GND
- removed copper zone on B.Cu, net (none)
- removed copper zone on F.Cu, net (none)
Other:
- board text added: "-"
- board text added: "DISK"
- board text added: "M1"
- board text added: "POWER"
- board text added: "PROG"
- board text added: "SuperEMUZ80 Rev 1.0 Feb 11, 2024 @hanyazou"
- board text removed: "SuperEMUZ80 Rev 0.9 Feb 3, 2024 @hanyazou"
