File: kicad/SuperEMUZ80.kicad_sch (KiCad schematic)
At the start: 31 parts, among them J1 EMUZ80_0, J2 EMUZ80, J4 Conn_02x01, J6 SD Card slot, J7 SD Card slot, U1 Z80CPU, U2 AS6C4008

Commit message: Add SuperEMUZ80 version 0.9
Parts:
- removed C1, C4: 100nF, Capacitor_THT:C_Disc_D4.3mm_W1.9mm_P5.00mm, symbol Device:C
- removed C5, C8: 100nF, Capacitor_SMD:C_0603_1608Metric_Pad1.08x0.95mm_HandSolder, symbol Device:C
- removed J1: EMUZ80_0, Connector_PinHeader_2.54mm:PinHeader_1x20_P2.54mm_Vertical, symbol library:EMUZ80_0
- removed J2: EMUZ80, Connector_PinHeader_2.54mm:PinHeader_1x20_P2.54mm_Vertical, symbol library:EMUZ80_1
- added C1, C3, C5, C7: 0.1uF, Capacitor_THT:C_Disc_D4.3mm_W1.9mm_P5.00mm, symbol Device:C_Small
- added C2, C4, C6, C8: 0.1uF, Capacitor_SMD:C_0603_1608Metric_Pad1.08x0.95mm_HandSolder, symbol Device:C_Small
- added D4: 1N4148, Diode_THT:D_DO-35_SOD27_P7.62mm_Horizontal, symbol Diode:1N4148
- added D7: DISK, LED_SMD:LED_0805_2012Metric_Pad1.15x1.40mm_HandSolder, symbol Device:LED
- added D8: M1, LED_SMD:LED_0805_2012Metric_Pad1.15x1.40mm_HandSolder, symbol Device:LED
- added D9: POWER, LED_SMD:LED_0805_2012Metric_Pad1.15x1.40mm_HandSolder, symbol Device:LED
- added J11: Conn_02x01, Connector_PinHeader_2.54mm:PinHeader_1x02_P2.54mm_Vertical, symbol Connector_Generic:Conn_02x01
- added J2: Conn_01x08_Pin, Connector_PinHeader_2.54mm:PinHeader_1x08_P2.54mm_Horizontal, symbol Connector:Conn_01x08_Pin
- added R16, R23, R31: 10K, Resistor_THT:R_Axial_DIN0204_L3.6mm_D1.6mm_P7.62mm_Horizontal, symbol Device:R
- added R17, R33: 10K, Resistor_SMD:R_0603_1608Metric_Pad0.98x0.95mm_HandSolder, symbol Device:R
- added R30: 40K, Resistor_THT:R_Axial_DIN0204_L3.6mm_D1.6mm_P7.62mm_Horizontal, symbol Device:R
- added R32: 40K, Resistor_SMD:R_0603_1608Metric_Pad0.98x0.95mm_HandSolder, symbol Device:R
- added S1: DTS-6, library:DTS-6, symbol library:DTS-6
- added S2: POWER, library:SS22F06, symbol mylib:slide_SW_big
- added U2: 18F47Q43, Package_DIP:DIP-40_W15.24mm_Socket, symbol mylib:PIC18F47Q43
- D1, D2, D3: footprint LED_THT:LED_D1.8mm_W3.3mm_H2.4mm -> LED_THT:LED_D5.0mm
- U1: footprint Package_DIP:DIP-40_W15.24mm -> Package_DIP:DIP-40_W15.24mm_Socket
- renumbered J4 to J1, J6 to J3, J7 to J4, R7 to R1, R1 to R10, R4 to R11, R2 to R12, R5 to R13, R3 to R14, R6 to R15, R8 to R2, R15 to R22, R9 to R3, R10 to R4, R11 to R5, R12 to R6, R13 to R7, R14 to R8, U2 to U3
Connections:
- net A0: now also U2.33 (RB0)
- net A1: now also U2.34 (RB1)
- net A14: now also U2.29 (RD6)
- net A15: now also U2.30 (RD7)
- net A16: now also U2.27 (RD4)
- net A17: now also U2.28 (RD5)
- net A2: now also U2.35 (RB2)
- net A3: now also U2.36 (RB3)
- net A4: now also U2.37 (RB4)
- net A5: now also U2.38 (RB5)
- net A6: now also J2.5 (Pin_5), U2.39 (RB6/ICSPC)
- net A7: now also J2.4 (Pin_4), U2.40 (RB7/ICSPD)
- net D0: now also U2.15 (RC0)
- net D1: now also U2.16 (RC1)
- net D2: now also U2.17 (RC2)
- net D3: now also U2.18 (RC3)
- net D4: now also U2.23 (RC4)
- net D5: now also U2.24 (RC5)
- net D6: now also U2.25 (RC6)
- net D7: now also U2.26 (RC7)
- net GND: now also C1.2, C2.2, C3.2, C4.2, C5.2, C6.2, C7.2, C8.2, D9.1 (K), J2.3 (Pin_3), R23.2, R30.2, R32.2, S1.3, S1.4, U2.12 (VSS), U2.31 (VSS)
- net MISO: now also U2.22 (RD3)
- net MOSI: now also U2.20 (RD1)
- net SCK: now also U2.21 (RD2)
- net ~{BUSRQ}: now also U2.4 (RA2)
- net ~{IORQ}: now also U2.2 (RA0)
- net ~{M1}: now also D8.1 (K)
- net ~{NMI}: now also R30.1, R31.2, R32.1, R33.2, U2.10 (RE2)
- net ~{RESET}: now also R23.1, U2.9 (RE1)
- net ~{SS}: now also D7.1 (K), U2.19 (RD0)
- net ~{WAIT}: now also U2.6 (RA4)
- net at D3.2 (A), R14.2, R15.2: now also D9.2 (A)
- net at D2.2 (A), R12.2, R13.2: now also D8.2 (A)
- net at D1.2 (A), R10.2, R11.2: now also D7.2 (A)
- net +5V renamed VCC
- net VCC: now also C1.1, C2.1, C3.1, C4.1, C5.1, C6.1, C7.1, C8.1, J2.2 (Pin_2), R16.1, R17.1, R31.1, R33.1, S2.1 (1A1), S2.6 (2A1), U2.11 (VDD), U2.32 (VDD)
- net RA3 renamed CLK_GEN
- net CLK_GEN: now also U2.5 (RA3)
- net ~{CE} renamed ~{MREQ}
- net ~{MREQ}: now also U2.3 (RA1)
- net ~{OE} renamed ~{RD}
- net ~{RD}: now also U2.7 (RA5)
- net ~{WE} renamed ~{WR}
- net ~{WR}: now also U2.8 (RE0)
- new net: D4.1 (K), J2.7 (Pin_7)
- new net PIC_RX: D4.2 (A), J11.2 (Pin_2), R16.2, R17.2, U2.13 (RA7)
- new net TX: J2.8 (Pin_8), U2.14 (RA6)
- new net picprog/PROG_TX: J11.1 (Pin_1)
- new net picprog/VDD: S2.2 (1A2), S2.5 (2A2)
- new net ~{MCLR}: J2.1 (Pin_1), S1.1, S1.2, U2.1 (~{MCLR}/RE3)
- no-connect marks 7 -> 6
Other:
- added sheet picprog (picprog.kicad_sch)
- note added: "Board ID 4.0V"
- title: SuperMEZ80-CPM -> SuperEMUZ80
- moved on the sheet: D1, D2, J1, JP1, R1, R10, R11, R12, R13, R2, R22, R3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

Commit message: Add SuperEMUZ80 version 1.0
Parts:
- D1, D7: value DISK -> LED
- D2, D8: value M1 -> LED
- D3, D9: value POWER -> LED
- R30, R32: value 40K -> 39K
Connections:
- net PIC_RX: no longer J11.2 (Pin_2)
- net at D4.1 (K), J2.7 (Pin_7): now also J11.2 (Pin_2)
Changed lines of the file:
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@@
   (title_block
     (title "SuperEMUZ80")
-    (date "2024-01-28")
-    (rev "0.9")
+    (date "2024-02-11")
+    (rev "1.0")
   )
   (junction (at 260.35 50.8) (diameter 0) (color 0 0 0 0)
@@
   (junction (at 260.35 55.88) (diameter 0) (color 0 0 0 0)
   )
+  (junction (at 190.5 149.86) (diameter 0) (color 0 0 0 0)
+  )
   (junction (at 196.85 120.65) (diameter 0) (color 0 0 0 0)
   )
@@
     (stroke (width 0) (type default))
   )
-  (wire (pts (xy 153.67 165.1) (xy 161.29 165.1))
-    (stroke (width 0) (type default))
-  )
   (wire (pts (xy 120.65 137.16) (xy 123.19 137.16))
     (stroke (width 0) (type default))
@@
     (stroke (width 0) (type default))
   )
+  (wire (pts (xy 190.5 149.86) (xy 190.5 165.1))
+    (stroke (width 0) (type default))
+  )
   (wire (pts (xy 45.72 172.72) (xy 52.07 172.72))
     (stroke (width 0) (type default))
@@
     (stroke (width 0) (type default))
   )
-  (wire (pts (xy 186.69 149.86) (xy 204.47 149.86))
+  (wire (pts (xy 186.69 149.86) (xy 190.5 149.86))
     (stroke (width 0) (type default))
   )
@@
     (stroke (width 0) (type default))
   )
+  (wire (pts (xy 190.5 149.86) (xy 204.47 149.86))
+    (stroke (width 0) (type default))
+  )
   (wire (pts (xy 228.6 142.24) (xy 233.68 142.24))
     (stroke (width 0) (type default))
@@
     (stroke (width 0) (type default))
   )
+  (wire (pts (xy 153.67 165.1) (xy 190.5 165.1))
+    (stroke (width 0) (type default))
+  )
   (bus (pts (xy 91.44 72.39) (xy 91.44 69.85))
     (stroke (width 0) (type default))
@@
     )
   )
-  (global_label "PIC_RX" (shape output) (at 161.29 165.1 0) (fields_autoplaced)
-    (effects (font (size 1.27 1.27)) (justify left))
-    (property "Intersheetrefs" "${INTERSHEET_REFS}" (at 170.7877 165.1 0)
-      (effects (font (size 1.27 1.27)) (justify left) hide)
-    )
-  )
   (global_label "A14" (shape input) (at 201.93 55.88 180) (fields_autoplaced)
     (effects (font (size 1.27 1.27)) (justify right))
@@
       (effects (font (size 1.27 1.27)))
     )
-    (property "Value" "POWER" (at 247.3325 120.65 0)
+    (property "Value" "LED" (at 247.3325 120.65 0)
       (effects (font (size 1.27 1.27)))
     )
@@
       (effects (font (size 1.27 1.27)))
     )
-    (property "Value" "M1" (at 247.3325 95.25 0)
+    (property "Value" "LED" (at 247.3325 95.25 0)
       (effects (font (size 1.27 1.27)))
     )
@@
       (effects (font (size 1.27 1.27)) (justify left))
     )
-    (property "Value" "40K" (at 209.55 36.195 0)
+    (property "Value" "39K" (at 209.55 36.195 0)
       (effects (font (size 1.27 1.27)) (justify left))
     )
@@
       (effects (font (size 1.27 1.27)))
     )
-    (property "Value" "DISK" (at 207.9625 101.6 0)
+    (property "Value" "LED" (at 207.9625 101.6 0)
       (effects (font (size 1.27 1.27)) hide)
     )
@@
       (effects (font (size 1.27 1.27)))
     )
-    (property "Value" "DISK" (at 207.9625 95.25 0)
+    (property "Value" "LED" (at 207.9625 95.25 0)
       (effects (font (size 1.27 1.27)))
     )
@@
       (effects (font (size 1.27 1.27)))
     )
-    (property "Value" "POWER" (at 247.3325 127 0)
+    (property "Value" "LED" (at 247.3325 127 0)
       (effects (font (size 1.27 1.27)) hide)
     )
@@
       (effects (font (size 1.27 1.27)))
     )
-    (property "Value" "M1" (at 247.3325 101.6 0)
+    (property "Value" "LED" (at 247.3325 101.6 0)
       (effects (font (size 1.27 1.27)) hide)
     )
@@
       (effects (font (size 1.27 1.27)) (justify left))
     )
-    (property "Value" "40K" (at 218.44 36.195 0)
+    (property "Value" "39K" (at 218.44 36.195 0)
       (effects (font (size 1.27 1.27)) (justify left))
     )
