File: kicad/picprog.kicad_sch (KiCad schematic)
At the start: 26 parts, among them J1 UART, J3 FW update, J4 ICSP Programmer, J5 5077CR-16SMC2-BK-TR, J8 ZX62-B-5PA_33_, U1 PIC16F1454-IP

Commit message: Add SuperEMUZ80 version 1.0
Parts:
- added R9 (x2): 5k1, Resistor_SMD:R_0603_1608Metric_Pad0.98x0.95mm_HandSolder, symbol Device:R
- R7, R8: value 220 -> 100
Connections:
- net GND: now also R9.2, R9.2
- net at J5.A5 (CC1), R10.1: now also R9.1
- net at J5.B5 (CC2), R9.1: now also R9.1
Changed lines of the file:
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@@
   (title_block
     (title "PIC Programmer 16F1454 (on-board)")
-    (date "2024-01-28")
+    (date "2024-02-11")
   )
   (junction (at 100.33 158.75) (diameter 0) (color 0 0 0 0)
@@
   (junction (at 102.87 120.65) (diameter 0) (color 0 0 0 0)
   )
+  (junction (at 219.71 71.12) (diameter 0) (color 0 0 0 0)
+  )
   (junction (at 53.34 158.75) (diameter 0) (color 0 0 0 0)
   )
+  (junction (at 215.9 83.82) (diameter 0) (color 0 0 0 0)
+  )
   (junction (at 215.9 87.63) (diameter 0) (color 0 0 0 0)
   )
@@
   (junction (at 259.08 132.08) (diameter 0) (color 0 0 0 0)
   )
+  (junction (at 215.9 71.12) (diameter 0) (color 0 0 0 0)
+  )
   (junction (at 215.9 59.69) (diameter 0) (color 0 0 0 0)
   )
@@
   )
   (junction (at 60.96 173.99) (diameter 0) (color 0 0 0 0)
+  )
+  (junction (at 219.71 83.82) (diameter 0) (color 0 0 0 0)
   )
   (junction (at 154.94 166.37) (diameter 0) (color 0 0 0 0)
@@
     (stroke (width 0) (type default))
   )
+  (wire (pts (xy 228.6 73.66) (xy 228.6 71.12))
+    (stroke (width 0) (type default))
+  )
   (wire (pts (xy 87.63 118.11) (xy 87.63 120.65))
     (stroke (width 0) (type default))
@@
     (stroke (width 0) (type default))
   )
+  (wire (pts (xy 208.28 81.28) (xy 208.28 83.82))
+    (stroke (width 0) (type default))
+  )
   (wire (pts (xy 166.37 166.37) (xy 165.1 166.37))
     (stroke (width 0) (type default))
@@
     (stroke (width 0) (type default))
   )
-  (wire (pts (xy 215.9 64.77) (xy 215.9 73.66))
+  (wire (pts (xy 215.9 64.77) (xy 215.9 71.12))
     (stroke (width 0) (type default))
   )
@@
     (stroke (width 0) (type default))
   )
+  (wire (pts (xy 208.28 73.66) (xy 208.28 71.12))
+    (stroke (width 0) (type default))
+  )
   (wire (pts (xy 166.37 175.26) (xy 166.37 166.37))
     (stroke (width 0) (type default))
@@
     (stroke (width 0) (type default))
   )
+  (wire (pts (xy 219.71 71.12) (xy 219.71 67.31))
+    (stroke (width 0) (type default))
+  )
   (wire (pts (xy 82.55 120.65) (xy 87.63 120.65))
     (stroke (width 0) (type default))
@@
     (stroke (width 0) (type default))
   )
+  (wire (pts (xy 228.6 83.82) (xy 219.71 83.82))
+    (stroke (width 0) (type default))
+  )
   (wire (pts (xy 236.22 87.63) (xy 236.22 88.9))
     (stroke (width 0) (type default))
@@
     (stroke (width 0) (type default))
   )
+  (wire (pts (xy 215.9 83.82) (xy 215.9 87.63))
+    (stroke (width 0) (type default))
+  )
+  (wire (pts (xy 228.6 71.12) (xy 219.71 71.12))
+    (stroke (width 0) (type default))
+  )
   (wire (pts (xy 266.7 59.69) (xy 266.7 57.15))
     (stroke (width 0) (type default))
   )
-  (wire (pts (xy 215.9 81.28) (xy 215.9 87.63))
+  (wire (pts (xy 215.9 81.28) (xy 215.9 83.82))
     (stroke (width 0) (type default))
   )
@@
     (stroke (width 0) (type default))
   )
+  (wire (pts (xy 208.28 83.82) (xy 215.9 83.82))
+    (stroke (width 0) (type default))
+  )
   (wire (pts (xy 110.49 170.18) (xy 110.49 173.99))
     (stroke (width 0) (type default))
   )
-  (wire (pts (xy 219.71 73.66) (xy 219.71 67.31))
+  (wire (pts (xy 219.71 73.66) (xy 219.71 71.12))
     (stroke (width 0) (type default))
   )
@@
     (stroke (width 0) (type default))
   )
+  (wire (pts (xy 219.71 83.82) (xy 219.71 87.63))
+    (stroke (width 0) (type default))
+  )
   (wire (pts (xy 100.33 158.75) (xy 100.33 165.1))
     (stroke (width 0) (type default))
   )
+  (wire (pts (xy 215.9 71.12) (xy 215.9 73.66))
+    (stroke (width 0) (type default))
+  )
   (wire (pts (xy 226.06 46.99) (xy 226.06 39.37))
     (stroke (width 0) (type default))
@@
     (stroke (width 0) (type default))
   )
+  (wire (pts (xy 208.28 71.12) (xy 215.9 71.12))
+    (stroke (width 0) (type default))
+  )
   (wire (pts (xy 226.06 62.23) (xy 215.9 62.23))
     (stroke (width 0) (type default))
@@
     (stroke (width 0) (type default))
   )
-  (wire (pts (xy 219.71 81.28) (xy 219.71 87.63))
+  (wire (pts (xy 219.71 81.28) (xy 219.71 83.82))
     (stroke (width 0) (type default))
   )
@@
   )
   (wire (pts (xy 246.38 96.52) (xy 246.38 97.79))
+    (stroke (width 0) (type default))
+  )
+  (wire (pts (xy 228.6 81.28) (xy 228.6 83.82))
     (stroke (width 0) (type default))
   )
@@
         (path "/d0b67a06-521c-429c-b0a7-be22c54278d6/7450f2a1-db01-4f25-b76e-d48b7f840353"
           (reference "R19") (unit 1)
+        )
+      )
+    )
+  )
+  (symbol (lib_id "Device:R") (at 228.6 77.47 0) (mirror y) (unit 1)
+    (in_bom yes) (on_board yes) (dnp no)
+    (property "Reference" "R9" (at 234.95 76.2 0)
+      (effects (font (size 1.27 1.27)) (justify left))
+    )
+    (property "Value" "5k1" (at 234.95 78.74 0)
+      (effects (font (size 1.27 1.27)) (justify left))
+    )
+    (property "Footprint" "Resistor_SMD:R_0603_1608Metric_Pad0.98x0.95mm_HandSolder" (at 230.378 77.47 90)
+      (effects (font (size 1.27 1.27)) hide)
+    )
+    (property "Datasheet" "~" (at 228.6 77.47 0)
+      (effects (font (size 1.27 1.27)) hide)
+    )
+    (pin "1")
+    (pin "2")
+    (instances
+      (project "picprog"
+        (path "/66c98a20-f61d-4a40-b4f3-4dc77024e47f"
+          (reference "R9") (unit 1)
+        )
+      )
+      (project "SuperEMUZ80"
+        (path "/d0b67a06-521c-429c-b0a7-be22c54278d6/7450f2a1-db01-4f25-b76e-d48b7f840353"
+          (reference "R35") (unit 1)
         )
       )
@@
         (path "/d0b67a06-521c-429c-b0a7-be22c54278d6/7450f2a1-db01-4f25-b76e-d48b7f840353"
           (reference "U4") (unit 1)
+        )
+      )
+    )
+  )
+  (symbol (lib_id "Device:R") (at 208.28 77.47 0) (mirror y) (unit 1)
+    (in_bom yes) (on_board yes) (dnp no)
+    (property "Reference" "R9" (at 205.74 76.835 0)
+      (effects (font (size 1.27 1.27)) (justify left))
+    )
+    (property "Value" "5k1" (at 205.74 79.375 0)
+      (effects (font (size 1.27 1.27)) (justify left))
+    )
+    (property "Footprint" "Resistor_SMD:R_0603_1608Metric_Pad0.98x0.95mm_HandSolder" (at 210.058 77.47 90)
+      (effects (font (size 1.27 1.27)) hide)
+    )
+    (property "Datasheet" "~" (at 208.28 77.47 0)
+      (effects (font (size 1.27 1.27)) hide)
+    )
+    (pin "1")
+    (pin "2")
+    (instances
+      (project "picprog"
+        (path "/66c98a20-f61d-4a40-b4f3-4dc77024e47f"
+          (reference "R9") (unit 1)
+        )
+      )
+      (project "SuperEMUZ80"
+        (path "/d0b67a06-521c-429c-b0a7-be22c54278d6/7450f2a1-db01-4f25-b76e-d48b7f840353"
+          (reference "R34") (unit 1)
         )
       )
@@
       (effects (font (size 1.27 1.27)))
     )
-    (property "Value" "220" (at 161.29 172.72 90)
+    (property "Value" "100" (at 161.29 172.72 90)
       (effects (font (size 1.27 1.27)))
     )
@@
       (effects (font (size 1.27 1.27)))
     )
-    (property "Value" "220" (at 161.29 163.83 90)
-      (effects (font (size 1.27 1.27)))
-    )
+    (property "Value" "100" (at 161.29 163.83 90)
+      (effects (font (size 1.27 1.27)))
+    )
